File: keyboard/keyboard.kicad_pcb (KiCad board)
At the start: 2 copper layers, 332.2 x 125.4 mm, 141 parts, among them SW1 SW_Push, SW10 SW_Push, SW11 SW_Push, SW12 SW_Push, SW13 SW_Push, SW14 SW_Push, SW15 SW_Push, SW16 SW_Push, SW17 SW_Push, SW18 SW_Push, SW19 SW_Push, SW2 SW_Push, SW20 SW_Push, SW21 SW_Push, SW22 SW_Push, SW23 SW_Push, SW24 SW_Push, SW25 SW_Push, SW26 SW_Push, SW27 SW_Push, SW28 SW_Push, SW29 SW_Push, SW3 SW_Push, SW30 SW_Push, SW32 SW_Push, SW33 SW_Push, SW34 SW_Push, SW35 SW_Push, SW36 SW_Push, SW37 SW_Push, SW38 SW_Push, SW39 SW_Push, SW4 SW_Push, SW40 SW_Push, SW41 SW_Push, SW42 SW_Push, SW43 SW_Push, SW44 SW_Push, SW45 SW_Push, SW46 SW_Push, SW47 SW_Push, SW48 SW_Push, SW49 SW_Push, SW5 SW_Push, SW50 SW_Push, SW51 SW_Push, SW52 SW_Push, SW53 SW_Push, SW54 SW_Push, SW55 SW_Push, SW56 SW_Push, SW57 SW_Push, SW58 SW_Push, SW59 SW_Push, SW6 SW_Push, SW60 SW_Push, SW61 SW_Push, SW62 SW_Push, SW63 SW_Push, SW64 SW_Push, SW65 SW_Push, SW66 SW_Push, SW67 SW_Push, SW7 SW_Push, SW8 SW_Push, SW9 SW_Push, U1 Elite-Pi-29-Pin-25-IO

Commit message: Updated keyboard project files
Parts:
- removed the REF** at (317.6, 7.26)
- removed the REF** at (277.7, 7.26)
- removed the Ref** at (261.3, 9.75)
- removed the Ref** at (302.1, 4.88)
- removed the Ref** at (261.4, 4.72)
- removed the Ref** at (302.0, 9.91)
- removed SW_Push: SW_31, PCM_Switch_Keyboard_Cherry_MX:SW_Cherry_MX_PCB_1.75u
- added EC11_Rotary_Encoder: RotaryEncoder_EC11, Keebio-Parts:RotaryEncoder_EC11, F.Cu at (313.0, 10.7)
- added EC11_Rotary_Encoder: RotaryEncoder_EC11, Keebio-Parts:RotaryEncoder_EC11, F.Cu at (270.4, 10.7)
- added LED_PAD: WS2812B SMD Strip 3mm, Library:WS2812B SMD Strip 3mm, F.Cu at (20.2, 89.1)
- added LED_PAD: WS2812B SMD Strip 3mm, Library:WS2812B SMD Strip 3mm, F.Cu at (20.1, 108.1)
- added LED_PAD: WS2812B SMD Strip 3mm, Library:WS2812B SMD Strip 3mm, F.Cu at (20.3, 70.0)
- added LED_PAD: WS2812B SMD Strip 3mm, Library:WS2812B SMD Strip 3mm, F.Cu at (20.3, 51.0)
- added REF**: WS2812B SMD Strip 3mm, Library:WS2812B SMD Strip 3mm, F.Cu at (20.1, 127.2)
- added Ref**: 10k, Keebio-Parts:Resistor, F.Cu at (296.6, 13.2)
- added Ref**: 10k, Keebio-Parts:Resistor, F.Cu at (254.1, 8.15)
- added Ref**: 10k, Keebio-Parts:Resistor, F.Cu at (254.0, 13.2)
- added Ref**: 10k, Keebio-Parts:Resistor, F.Cu at (296.7, 8.17)
- added SW_31: SW_Push, PCM_Switch_Keyboard_Cherry_MX:SW_Cherry_MX_PCB_1.75u, F.Cu at (34.3, 76.0)
- added U4: HOLE, Keebio-Parts:MountingHole, F.Cu at (296.4, 21.2)
- added U4: HOLE, Keebio-Parts:MountingHole, F.Cu at (5.35, 114.7)
- added U4: HOLE, Keebio-Parts:MountingHole, F.Cu at (203.5, 114.9)
- added U4: HOLE, Keebio-Parts:MountingHole, F.Cu at (5.35, 69.5)
- U1: value Elite-Pi-29-Pin-25-IO -> Elite-C; footprint Keebio-Parts:Elite-C-castellated-29pin-holes -> Keebio-Parts:Elite-C
- moved D65 8.11 mm to (279.9, 117.2)
- moved D66 8.11 mm to (299.0, 117.2)
- moved D67 8.11 mm to (318.0, 117.2)
- moved SW65 8.11 mm to (274.8, 114.2)
- moved SW66 8.11 mm to (293.9, 114.2)
- moved D25 8.11 mm to (213.2, 60.0)
- moved D28 8.11 mm to (270.4, 60.0)
- moved D29 8.11 mm to (294.2, 60.0)
- moved D30 8.11 mm to (318.0, 60.0)
- moved SW9 8.11 mm to (179.6, 38.0)
- moved D15 8.11 mm to (318.0, 41.0)
- moved D36 8.11 mm to (141.8, 79.1)
- moved D41 8.11 mm to (237.0, 79.1)
- moved D42 8.11 mm to (256.1, 79.1)
- moved D43 8.11 mm to (287.0, 79.1)
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Connections:
- U1 pad 1: (no net) -> A_OUT_R
- U1 pad 10: COL2 -> COL1
- U1 pad 11: COL3 -> COL2
- U1 pad 12: COL4 -> COL3
- U1 pad 13: COL10 -> COL9
- U1 pad 14: ROW1 -> ROW4
- U1 pad 15: ROW2 -> ROW1
- U1 pad 17: ROW4 -> ROW2
- U1 pad 18: ROW5 -> ROW6
- U1 pad 19: ROW6 -> ROW5
- U1 pad 2: (no net) -> B_OUT_R
- U1 pad 24: (no net) -> COL10
- U1 pad 25: COL5 -> COL4
- U1 pad 26: COL6 -> COL5
- U1 pad 27: COL7 -> COL6
- U1 pad 28: COL8 -> COL7
- U1 pad 29: COL9 -> COL8
- U1 pad 3: SWR -> (no net)
- U1 pad 4: BR -> GND_LED
- U1 pad 5: AR -> SW_R
- U1 pad 6: SW -> DIN
- U1 pad 7: BL -> A_OUT
- U1 pad 8: AL -> B_OUT
- U1 pad 9: COL1 -> SW
Routing:
- net ROW6: track 796.2 -> 0.00 mm
- net COL2: track 706.5 -> 0.00 mm
- net ROW4: track 702.9 -> 0.00 mm
- net COL3: track 683.2 -> 0.00 mm
- net COL1: track 671.1 -> 0.00 mm
- net COL4: track 668.8 -> 0.00 mm
- net ROW7: track 655.1 -> 0.00 mm
- net COL5: track 638.8 -> 0.00 mm
- net COL7: track 556.0 -> 0.00 mm
- net COL8: track 554.6 -> 0.00 mm
- net COL9: track 535.5 -> 0.00 mm
- net ROW5: track 523.4 -> 0.00 mm
- net ROW3: track 490.9 -> 0.00 mm
- net COL10: track 432.4 -> 0.00 mm
- net ROW1: track 403.6 -> 0.00 mm
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Other:
- board size 332.2 x 125.4 mm -> 332.3 x 125.9 mm
- board text added: "B0"
- board text added: "B1"
- board text added: "B2"
- board text added: "B3"
- board text added: "B4"
- board text added: "B5"
- board text added: "B6"
- board text added: "B7"
- board text added: "C6"
- board text added: "C7"
- board text added: "D0"
- board text added: "D1"
- board text added: "D2"
- board text added: "D4"
- board text added: "D5"
- board text added: "D7"
- board text added: "E6"
- board text added: "F0"
- board text added: "F1"
- board text added: "F4"
- board text added: "F5"
- board text added: "F6"
- board text added: "F7"
- board text added: "GND"
- board text added: "LED_PAD"
- board text added: "ST"
- board text added: "VCC"
