File: keyboard/keyboard.kicad_pcb (KiCad board)
At the start: 2 copper layers, 332.3 x 125.9 mm, 150 parts, among them SW1 SW_Push, SW10 SW_Push, SW11 SW_Push, SW12 SW_Push, SW13 SW_Push, SW14 SW_Push, SW15 SW_Push, SW16 SW_Push, SW17 SW_Push, SW18 SW_Push, SW19 SW_Push, SW2 SW_Push, SW20 SW_Push, SW21 SW_Push, SW22 SW_Push, SW23 SW_Push, SW24 SW_Push, SW25 SW_Push, SW26 SW_Push, SW27 SW_Push, SW28 SW_Push, SW29 SW_Push, SW3 SW_Push, SW30 SW_Push, SW32 SW_Push, SW33 SW_Push, SW34 SW_Push, SW35 SW_Push, SW36 SW_Push, SW37 SW_Push, SW38 SW_Push, SW39 SW_Push, SW4 SW_Push, SW40 SW_Push, SW41 SW_Push, SW42 SW_Push, SW43 SW_Push, SW44 SW_Push, SW45 SW_Push, SW46 SW_Push, SW47 SW_Push, SW48 SW_Push, SW49 SW_Push, SW5 SW_Push, SW50 SW_Push, SW51 SW_Push, SW52 SW_Push, SW53 SW_Push, SW54 SW_Push, SW55 SW_Push, SW56 SW_Push, SW57 SW_Push, SW58 SW_Push, SW59 SW_Push, SW6 SW_Push, SW60 SW_Push, SW61 SW_Push, SW62 SW_Push, SW63 SW_Push, SW64 SW_Push, SW65 SW_Push, SW66 SW_Push, SW67 SW_Push, SW7 SW_Push, SW8 SW_Push, SW9 SW_Push, U1 Elite-C, U4 HOLE

Commit message: started working on traces,
Im not 100% on the pcb design so I may go into ergogen and mess around with it
Parts:
- moved D42 176.7 mm to (367.3, 216.4)
- moved D65 176.7 mm to (391.2, 254.5)
- moved D1 176.7 mm to (143.5, 178.3)
- moved D11 176.7 mm to (334.0, 178.3)
- moved D12 176.7 mm to (353.1, 178.3)
- moved D13 176.7 mm to (372.1, 178.3)
- moved D14 176.7 mm to (400.7, 178.3)
- moved D15 176.7 mm to (429.3, 178.3)
- moved D16 176.7 mm to (148.3, 197.3)
- moved D17 176.7 mm to (172.1, 197.3)
- moved D18 176.7 mm to (191.1, 197.3)
- moved D19 176.7 mm to (210.2, 197.3)
- moved D2 176.7 mm to (162.6, 178.3)
- moved D20 176.7 mm to (229.2, 197.3)
- moved D21 176.7 mm to (248.3, 197.3)
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Routing:
- net N$67: track 0.00 -> 10.8 mm
- net N$28: track 0.00 -> 10.1 mm
- net N$30: track 0.00 -> 9.91 mm
- net N$15: track 0.00 -> 9.91 mm
- net N$26: track 0.00 -> 9.82 mm
- net N$23: track 0.00 -> 9.79 mm
- net N$24: track 0.00 -> 9.64 mm
- net N$29: track 0.00 -> 9.08 mm
- net N$27: track 0.00 -> 9.08 mm
- net N$25: track 0.00 -> 9.08 mm
- net N$38: track 0.00 -> 8.22 mm
- net N$62: track 0.00 -> 8.18 mm
- net N$20: track 0.00 -> 8.06 mm
- net N$17: track 0.00 -> 8.06 mm
- net N$16: track 0.00 -> 8.06 mm
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